File: buckBoost.kicad_sch (KiCad schematic)
At the start: 16 parts

Commit message: V2 adds a power switch
Parts:
- C101, C102, C105, C106, C107: value (none) -> 10u; footprint (none) -> Capacitor_SMD:C_0805_2012Metric_Pad1.15x1.40mm_HandSolder
- C103: value (none) -> 0.1u; footprint (none) -> Capacitor_SMD:C_0805_2012Metric_Pad1.15x1.40mm_HandSolder
- C104: value (none) -> 10p; footprint (none) -> Capacitor_SMD:C_0805_2012Metric_Pad1.15x1.40mm_HandSolder
- C108: value (none) -> C; footprint (none) -> Capacitor_SMD:C_0805_2012Metric_Pad1.15x1.40mm_HandSolder
- D101: value (none) -> LED; footprint (none) -> Diode_SMD:D_0805_2012Metric_Pad1.15x1.40mm_HandSolder
- L101: value (none) -> LPS4020-152; footprint (none) -> Inductor_SMD:L_Coilcraft_XxL4020
- R101: value (none) -> 1M; footprint (none) -> Resistor_SMD:R_0805_2012Metric_Pad1.15x1.40mm_HandSolder
- R102: value (none) -> 180k; footprint (none) -> Resistor_SMD:R_0805_2012Metric_Pad1.15x1.40mm_HandSolder
- R103: value (none) -> 1k; footprint (none) -> Diode_SMD:D_0805_2012Metric_Pad1.15x1.40mm_HandSolder
- SW1: value (none) -> PWRON; footprint (none) -> Button_Switch_SMD:SW_SPDT_PCM12
- U101: value (none) -> BUCKBOOST; footprint (none) -> Accelerando:BUCKBOOST
- U102: value (none) -> TPS63060; footprint (none) -> Package_SON:Texas_S-PWSON-N10_ThermalVias
